File: hardware/stay-awake-v1/stay-awake-v1.sch (KiCad schematic (older format))
At the start: 12 parts, among them J1 USB_A, U1 ATtiny85-20PU, Y1 16MHz

Commit message: Add pcb
Parts:
- C1, C2: footprint (none) -> Capacitors_THT:C_Disc_D3.0mm_W1.6mm_P2.50mm
- C3: footprint (none) -> Capacitors_THT:C_Disc_D5.0mm_W2.5mm_P5.00mm
- C4: footprint (none) -> Capacitors_THT:CP_Radial_Tantal_D5.0mm_P2.50mm
- D1, D2: footprint (none) -> Diodes_THT:D_A-405_P7.62mm_Horizontal
- J1: footprint (none) -> Connectors:USB_A
- R1, R2, R3: footprint (none) -> Resistors_THT:R_Axial_DIN0207_L6.3mm_D2.5mm_P7.62mm_Horizontal
- Y1: footprint (none) -> Crystals:Resonator-2pin_w8.0mm_h3.5mm
Changed lines of the file:
@@
 F 0 "J1" H 3370 1589 50  0000 R CNN
 F 1 "USB_A" H 3370 1498 50  0000 R CNN
-F 2 "" H 3750 1550 50  0001 C CNN
+F 2 "Connectors:USB_A" H 3750 1550 50  0001 C CNN
 F 3 " ~" H 3750 1550 50  0001 C CNN
 	1    3600 1600
@@
 F 0 "R1" V 2600 1600 50  0000 C CNN
 F 1 "68R" V 2500 1600 50  0000 C CNN
-F 2 "" V 2430 1600 50  0001 C CNN
+F 2 "Resistors_THT:R_Axial_DIN0207_L6.3mm_D2.5mm_P7.62mm_Horizontal" V 2430 1600 50  0001 C CNN
 F 3 "" H 2500 1600 50  0001 C CNN
 	1    2500 1600
@@
 F 0 "R2" V 2600 1800 50  0000 C CNN
 F 1 "68R" V 2500 1800 50  0000 C CNN
-F 2 "" V 2430 1800 50  0001 C CNN
+F 2 "Resistors_THT:R_Axial_DIN0207_L6.3mm_D2.5mm_P7.62mm_Horizontal" V 2430 1800 50  0001 C CNN
 F 3 "" H 2500 1800 50  0001 C CNN
 	1    2500 1800
@@
 F 0 "R3" V 2400 2100 50  0000 C CNN
 F 1 "2k2" V 2500 2100 50  0000 C CNN
-F 2 "" V 2430 2100 50  0001 C CNN
+F 2 "Resistors_THT:R_Axial_DIN0207_L6.3mm_D2.5mm_P7.62mm_Horizontal" V 2430 2100 50  0001 C CNN
 F 3 "" H 2500 2100 50  0001 C CNN
 	1    2500 2100
@@
 F 0 "D1" V 2854 2129 50  0000 L CNN
 F 1 "3v6" V 2945 2129 50  0000 L CNN
-F 2 "" H 2900 2050 50  0001 C CNN
+F 2 "Diodes_THT:D_A-405_P7.62mm_Horizontal" H 2900 2050 50  0001 C CNN
 F 3 "https://en.wikipedia.org/wiki/Zener_diode" H 2900 2050 50  0001 C CNN
 	1    2900 2050
@@
 F 0 "D2" V 3154 2129 50  0000 L CNN
 F 1 "3v6" V 3245 2129 50  0000 L CNN
-F 2 "" H 3200 2050 50  0001 C CNN
+F 2 "Diodes_THT:D_A-405_P7.62mm_Horizontal" H 3200 2050 50  0001 C CNN
 F 3 "https://en.wikipedia.org/wiki/Zener_diode" H 3200 2050 50  0001 C CNN
 	1    3200 2050
@@
 F 0 "Y1" V 2554 1488 50  0000 L CNN
 F 1 "16MHz" V 2600 1300 50  0000 L CNN
-F 2 "" H 2600 1400 50  0001 C CNN
+F 2 "Crystals:Resonator-2pin_w8.0mm_h3.5mm" H 2600 1400 50  0001 C CNN
 F 3 "" H 2600 1400 50  0001 C CNN
 	1    2600 1400
@@
 F 0 "C2" H 3042 1446 50  0000 L CNN
 F 1 "22pF" H 3042 1355 50  0000 L CNN
-F 2 "" H 2950 1400 50  0001 C CNN
+F 2 "Capacitors_THT:C_Disc_D3.0mm_W1.6mm_P2.50mm" H 2950 1400 50  0001 C CNN
 F 3 "" H 2950 1400 50  0001 C CNN
 	1    2950 1400
@@
 F 0 "C1" H 2592 1146 50  0000 L CNN
 F 1 "22pF" H 2592 1055 50  0000 L CNN
-F 2 "" H 2500 1100 50  0001 C CNN
+F 2 "Capacitors_THT:C_Disc_D3.0mm_W1.6mm_P2.50mm" H 2500 1100 50  0001 C CNN
 F 3 "" H 2500 1100 50  0001 C CNN
 	1    2500 1100
@@
 F 0 "C3" H 1765 2396 50  0000 L CNN
 F 1 "100n" H 1765 2305 50  0000 L CNN
-F 2 "" H 1688 2200 50  0001 C CNN
+F 2 "Capacitors_THT:C_Disc_D5.0mm_W2.5mm_P5.00mm" H 1688 2200 50  0001 C CNN
 F 3 "" H 1650 2350 50  0001 C CNN
 	1    1650 2350
@@
 F 0 "C4" H 2168 2396 50  0000 L CNN
 F 1 "10u" H 2168 2305 50  0000 L CNN
-F 2 "" H 2088 2200 50  0001 C CNN
+F 2 "Capacitors_THT:CP_Radial_Tantal_D5.0mm_P2.50mm" H 2088 2200 50  0001 C CNN
 F 3 "" H 2050 2350 50  0001 C CNN
 	1    2050 2350
